Commit message: Add files via upload

File: tinkerkit_description/urdf/tinkerkit.urdf (robot description, URDF)
Before this commit: robot tinkerkit, 9 links, 8 joints
Links:
- link arm_link: geometry collision mesh filename=file:/home/binn/robot_ws/tinkerkit/src/tinkerkit_descriptio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 scale=0.001 0.001 0.001; visual mesh filename=file:/home/binn/robot_ws/tinkerkit/src/tinkerkit_descriptio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 scale=0.001 0.001 0.001
- link base_link: geometry collision mesh filename=file:/home/binn/robot_ws/tinkerkit/src/tinkerkit_descriptio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 scale=0.001 0.001 0.001; visual mesh filename=file:/home/binn/robot_ws/tinkerkit/src/tinkerkit_descriptio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 scale=0.001 0.001 0.001
- link elbow_link: geometry collision mesh filename=file:/home/binn/robot_ws/tinkerkit/src/tinkerkit_descriptio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 scale=0.001 0.001 0.001; visual mesh filename=file:/home/binn/robot_ws/tinkerkit/src/tinkerkit_descriptio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 scale=0.001 0.001 0.001
- link hand_link: geometry collision mesh filename=file:/home/binn/robot_ws/tinkerkit/src/tinkerkit_descriptio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 scale=0.001 0.001 0.001; visual mesh filename=file:/home/binn/robot_ws/tinkerkit/src/tinkerkit_descriptio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 scale=0.001 0.001 0.001
- link left_gripper: geometry collision mesh filename=file:/home/binn/robot_ws/tinkerkit/src/tinkerkit_descriptio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 scale=0.001 0.001 0.001; visual mesh filename=file:/home/binn/robot_ws/tinkerkit/src/tinkerkit_descriptio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 scale=0.001 0.001 0.001
- link right_gripper: geometry collision mesh filename=file:/home/binn/robot_ws/tinkerkit/src/tinkerkit_descriptio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 scale=0.001 0.001 0.001; visual mesh filename=file:/home/binn/robot_ws/tinkerkit/src/tinkerkit_descriptio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 scale=0.001 0.001 0.001
- link shoulder_link: geometry collision mesh filename=file:/home/binn/robot_ws/tinkerkit/src/tinkerkit_descriptio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 scale=0.001 0.001 0.001; visual mesh filename=file:/home/binn/robot_ws/tinkerkit/src/tinkerkit_descriptio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 scale=0.001 0.001 0.001
- link wrist_link: geometry collision mesh filename=file:/home/binn/robot_ws/tinkerkit/src/tinkerkit_descriptio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 scale=0.001 0.001 0.001; visual mesh filename=file:/home/binn/robot_ws/tinkerkit/src/tinkerkit_descriptio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 scale=0.001 0.001 0.001
